File: hardware/rf-power-detector.brd (EAGLE design)
At the start: 44 x 29 mm, 37 parts, among them U1 AD8317, U4 MIC5301

Commit message: hw: add a 150Ohm load on the adc input
Parts:
- R10: value dnp -> 150
Changed lines of the file:
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@@
 <element name="LP1" library="balto" package="VLP-XXX-X" value="VLP-XXX-X" x="22.2504" y="24.6888" rot="R180"/>
 <element name="R1" library="rcl" package="R0603" value="52.3" x="24.6888" y="13.5636" rot="R90"/>
-<element name="R10" library="rcl" package="R0603" value="dnp" x="12.8016" y="12.192" rot="R90"/>
+<element name="R10" library="rcl" package="R0603" value="150" x="12.8016" y="12.192" rot="R90"/>
 <element name="R13" library="rcl" package="R0603" value="330" x="17.9832" y="23.9268" rot="R180"/>
 <element name="R15" library="rcl" package="R0603" value="330" x="17.9832" y="25.4508" rot="R180"/>
